Commit message: Update revolute.urdf
updating revolute urdf

File: src/udm_urdf/urdf/revolute.urdf (robot description, URDF)
Before this commit: robot human_hand, 13 links, 13 joints
Links:
- added link finger_one_link; visual cylinder length=0.0242 radius=0.01905
- added link finger_one_part_three_link; visual cylinder length=0.0242 radius=0.01905
- added link finger_one_part_two_link; visual cylinder length=0.0242 radius=0.01905
- added link finger_three_link; visual cylinder length=0.0242 radius=0.01905
- added link finger_three_part_three_link; visual cylinder length=0.0242 radius=0.01905
- added link finger_three_part_two_link; visual cylinder length=0.0242 radius=0.01905
- added link finger_two_link; visual cylinder length=0.0242 radius=0.01905
- added link finger_two_part_three_link; visual cylinder length=0.0242 radius=0.01905
- added link finger_two_part_two_link; visual cylinder length=0.0242 radius=0.01905
- added link forearm_link; visual cylinder length=0.0242 radius=0.01905
- added link forearm_revolute; visual cylinder length=0.0242 radius=0.01905
- added link thumb_2nd_part_joint_revolute; visual cylinder length=0.0242 radius=0.01905
- added link thumb_joint_revolute; visual cylinder length=0.0242 radius=0.01905
Joints:
- removed joint forearm_revolute
- added joint joint_2nd_part_thumb__revolute: type revolute, parent palm, child thumb_2nd_part_joint_revolute, origin xyz=0 0 0 rpy=0 0 0, axis 0 0 1, limit lower=-3.1416 upper=3.1416 effort=10 velocity=3
- added joint joint_finger_one: type revolute, parent palm, child finger_one_link, origin xyz=0 0 0.8 rpy=0 0 0, axis 0 0 1, limit lower=-3.1416 upper=3.1416 effort=10 velocity=3
- added joint joint_finger_one_part_three: type revolute, parent first_finger_part_two, child finger_one_part_three_link, origin xyz=0 0 0 rpy=0 0 0, axis 0 0 1, limit lower=-3.1416 upper=3.1416 effort=10 velocity=3
- added joint joint_finger_one_part_two: type revolute, parent first_finger, child finger_one_part_two_link, origin xyz=0 0 0.8 rpy=0 0 0, axis 0 0 1, limit lower=-3.1416 upper=3.1416 effort=10 velocity=3
- added joint joint_finger_three: type revolute, parent palm, child finger_three_link, origin xyz=0 0 0.8 rpy=0 0 0, axis 0 0 1, limit lower=-3.1416 upper=3.1416 effort=10 velocity=3
- added joint joint_finger_three_part_three: type revolute, parent third_finger_part_three, child finger_three_part_three_link, origin xyz=0 0 0 rpy=0 0 0, axis 0 0 1, limit lower=-3.1416 upper=3.1416 effort=10 velocity=3
- added joint joint_finger_three_part_two: type revolute, parent third_finger, child finger_three_part_two_link, origin xyz=0 0 0.8 rpy=0 0 0, axis 0 0 1, limit lower=-3.1416 upper=3.1416 effort=10 velocity=3
- added joint joint_finger_two: type revolute, parent palm, child finger_two_link, origin xyz=0 0 0.8 rpy=0 0 0, axis 0 0 1, limit lower=-3.1416 upper=3.1416 effort=10 velocity=3
- added joint joint_finger_two_part_three: type revolute, parent second_finger_part_three, child finger_two_part_three_link, origin xyz=0 0 0 rpy=0 0 0, axis 0 0 1, limit lower=-3.1416 upper=3.1416 effort=10 velocity=3
- added joint joint_finger_two_part_two: type revolute, parent second_finger, child finger_two_part_two_link, origin xyz=0 0 0.8 rpy=0 0 0, axis 0 0 1, limit lower=-3.1416 upper=3.1416 effort=10 velocity=3
- added joint joint_forearm: type revolute, parent base_link, child forearm_link, origin xyz=0 0 0 rpy=0 0 0.4, axis 0 0 1, limit lower=-3.1416 upper=3.1416 effort=10 velocity=3
- added joint joint_forearm_revolute: type revolute, parent base_link, child forearm_revolute, origin xyz=0 0 0 rpy=0 0 0, axis 0 0 1, limit lower=-3.1416 upper=3.1416 effort=10 velocity=3
- added joint joint_thumb__revolute: type revolute, parent palm, child thumb_joint_revolute, origin xyz=0 0 0 rpy=0 0 0, axis 0 0 1, limit lower=-3.1416 upper=3.1416 effort=10 velocity=3

Commit message: Update revolute.urdf

File: src/udm_urdf/urdf/revolute.urdf (robot description, URDF)
Before this commit: robot human_hand, 26 links, 25 joints
Links:
- removed link finger_one_link
- removed link finger_one_part_three_link
- removed link finger_one_part_two_link
- removed link finger_three_link
- removed link finger_three_part_three_link
- removed link finger_three_part_two_link
- removed link finger_two_link
- removed link finger_two_part_three_link
- removed link finger_two_part_two_link
- removed link forearm_link
- removed link forearm_revolute
- removed link thumb_2nd_part_joint_revolute
- removed link thumb_joint_revolute
Joints:
- removed joint joint_2nd_part_thumb__revolute
- removed joint joint_finger_one
- removed joint joint_finger_one_part_three
- removed joint joint_finger_one_part_two
- removed joint joint_finger_three
- removed joint joint_finger_three_part_three
- removed joint joint_finger_three_part_two
- removed joint joint_finger_two
- removed joint joint_finger_two_part_three
- removed joint joint_finger_two_part_two
- removed joint joint_forearm
- removed joint joint_forearm_revolute
- removed joint joint_thumb__revolute
- added joint forearm_revolute: type revolute, parent base_link, child palm, origin xyz=0.0 0.0 0.4 rpy=0 0 0, axis  0 1 0, limit lower=-3.14 upper=3.14 effort=10 velocity=3
- joint finger_one: axis (none) -> 1 0 0; limit (none) -> lower=-1.0 upper=1.0 effort=1000.0 velocity=0.5; type fixed -> revolute
- joint finger_one_part_three: axis (none) -> 1 0 0; limit (none) -> lower=-0.5 upper=0 effort=1000.0 velocity=0.5; type fixed -> revolute
- joint finger_one_part_two: axis (none) -> 1 0 0; limit (none) -> lower=-1.0 upper=0 effort=1000.0 velocity=0.5; type fixed -> revolute
- joint finger_three: axis (none) -> 1 0 0; limit (none) -> lower=-1.0 upper=1.0 effort=1000.0 velocity=0.5; type fixed -> revolute
- joint finger_three_part_three: axis (none) -> 1 0 0; limit (none) -> lower=-1.0 upper=1.0 effort=1000.0 velocity=0.5; type fixed -> revolute
- joint finger_three_part_two: axis (none) -> 1 0 0; limit (none) -> lower=-1.0 upper=1.0 effort=1000.0 velocity=0.5; type fixed -> revolute
- joint finger_two: axis (none) -> 1 0 0; limit (none) -> lower=-1.0 upper=1.0 effort=1000.0 velocity=0.5; type fixed -> revolute
- joint finger_two_part_three: axis (none) -> 1 0 0; limit (none) -> lower=-1.0 upper=1.0 effort=1000.0 velocity=0.5; type fixed -> revolute
- joint finger_two_part_two: axis (none) -> 1 0 0; limit (none) -> lower=-1.0 upper=1.0 effort=1000.0 velocity=0.5; type fixed -> revolute
- joint part_two_thumb: axis (none) -> 1 0 0; limit (none) -> lower=-1.0 upper=1.0 effort=1000.0 velocity=0.5; type fixed -> revolute
- joint thumb_joint: axis (none) -> 1 0 0; limit (none) -> lower=-1.0 upper=1.0 effort=1000.0 velocity=0.5; type fixed -> revolute

Commit message: Update revolute.urdf
updating finger tips

File: src/udm_urdf/urdf/revolute.urdf (robot description, URDF)
Before this commit: robot human_hand, 13 links, 13 joints
Links:
- added link head_finger_one; visual sphere radius=0.05
- added link head_finger_three; visual sphere radius=0.05
- added link head_finger_two; visual sphere radius=0.05
- added link head_thumb; visual sphere radius=0.05
Joints:
- added joint head_finger_one_joint: type fixed, parent first_finger_part_three, child head_finger_one, origin xyz=0 0 0.2
- added joint head_finger_three_joint: type fixed, parent third_finger_part_three, child head_finger_three, origin xyz=0 0 0.2
- added joint head_finger_two_joint: type fixed, parent second_finger_part_three, child head_finger_two, origin xyz=0 0 0.2
- added joint head_thumb_joint: type fixed, parent thumb_part_two, child head_thumb, origin xyz=0.175 -0.02 0.1 rpy=0 0 0
- joint forearm_revolute: axis  0 1 0 ->  0 0 1
