Commit message: Update main.urdf

File: src/udm_urdf/urdf/main.urdf (robot description, URDF)
Before this commit: robot human_hand, 13 links, 12 joints
Joints:
- added joint forearm_revolute: type revolute, parent base_link, child palm, origin xyz=0.0 0.0 0.4 rpy=0 0 0, axis  1 0 0, limit lower=-3.14 upper=3.14 effort=10 velocity=3

Commit message: Update main.urdf

File: src/udm_urdf/urdf/main.urdf (robot description, URDF)
Before this commit: robot human_hand, 13 links, 13 joints
Joints:
- removed joint forearm_revolute

Commit message: Update main.urdf
Updating finger tips

File: src/udm_urdf/urdf/main.urdf (robot description, URDF)
Before this commit: robot human_hand, 13 links, 12 joints
Links:
- added link head_finger_one; visual sphere radius=0.05
- added link head_finger_three; visual sphere radius=0.05
- added link head_finger_two; visual sphere radius=0.05
- added link head_thumb; visual sphere radius=0.05
Joints:
- added joint head_finger_one_joint: type fixed, parent first_finger_part_three, child head_finger_one, origin xyz=0 0 0.2
- added joint head_finger_three_joint: type fixed, parent third_finger_part_three, child head_finger_three, origin xyz=0 0 0.2
- added joint head_finger_two_joint: type fixed, parent second_finger_part_three, child head_finger_two, origin xyz=0 0 0.2
- added joint head_thumb_joint: type fixed, parent thumb_part_two, child head_thumb, origin xyz=0.175 -0.02 0.1 rpy=0 0 0
